File: modules/audio-codec/audio-codec.kicad_sch (KiCad schematic)
At the start: 24 parts, among them U1 TLV320AIC3110IRHBR, U2 ADP5301ACBZ-1-R7

Commit message: Updating audio-codec
Parts:
- M1: footprint MegaCastle:MegaCastle2x11-Module-I17.7x23.1-MBFFFFC-PANEL-NIBBLE -> MegaCastle:MegaCastle2x11-Module-I22.0x23.1-MBFFFFC-SPAREPAD
- U1: footprint TLV320AIC3110IRHBR:IC_ADS125H01IRHBT -> audio-codec:IC_ADS125H01IRHBT
- U2: footprint BGA9C50P3X3_187X165X66N -> audio-codec:BGA9C50P3X3_187X165X66N
Changed lines of the file:
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@@
 (kicad_sch
-	(version 20231120)
+	(version 20250114)
 	(generator "eeschema")
-	(generator_version "8.0")
+	(generator_version "9.0")
 	(paper "A4")
+	(text "Pull SYNC/MODE high for\ndefault 500mA max, but\nat lower efficiency for\nlow current draw.\nExternal pad allows pulling\nit low (or clocking the PWM)\nif desired."
+		(exclude_from_sim no)
+		(at 13.716 54.61 0)
+		(effects
+			(font
+				(size 1.27 1.27)
+			)
+			(justify left)
+		)
+	)
+	(text "19.6K selects\n1.8V for -1-R7"
+		(exclude_from_sim no)
+		(at 41.402 74.168 0)
+		(effects
+			(font
+				(size 1.27 1.27)
+			)
+			(justify left)
+		)
+	)
+	(text "= +1.8V Rail"
+		(exclude_from_sim no)
+		(at 135.382 118.618 0)
+		(effects
+			(font
+				(size 1.27 1.27)
+			)
+			(justify right)
+		)
+	)
+	(text "DVSS & IOVSS tied to\ndigital side of GND\nplane.\n\nAll others to analog\n(VBAT) side."
+		(exclude_from_sim no)
+		(at 189.484 130.556 0)
+		(effects
+			(font
+				(size 1.27 1.27)
+			)
+			(justify left)
+		)
+	)
 	(junction
 		(at 267.97 53.34)
@@
 		)
 	)
-	(text "Pull SYNC/MODE high for\ndefault 500mA max, but\nat lower efficiency for\nlow current draw.\nExternal pad allows pulling\nit low (or clocking the PWM)\nif desired."
-		(exclude_from_sim no)
-		(at 13.716 54.61 0)
-		(effects
-			(font
-				(size 1.27 1.27)
-			)
-			(justify left)
-		)
-	)
-	(text "19.6K selects\n1.8V for -1-R7"
-		(exclude_from_sim no)
-		(at 41.402 74.168 0)
-		(effects
-			(font
-				(size 1.27 1.27)
-			)
-			(justify left)
-		)
-	)
-	(text "= +1.8V Rail"
-		(exclude_from_sim no)
-		(at 135.382 118.618 0)
-		(effects
-			(font
-				(size 1.27 1.27)
-			)
-			(justify right)
-		)
-	)
-	(text "DVSS & IOVSS tied to\ndigital side of GND\nplane.\n\nAll others to analog\n(VBAT) side."
-		(exclude_from_sim no)
-		(at 189.484 130.556 0)
-		(effects
-			(font
-				(size 1.27 1.27)
-			)
-			(justify left)
-		)
-	)
 	(global_label "3.5MM_MIC"
 		(shape input)
@@
 			)
 		)
-		(property "Footprint" "TLV320AIC3110IRHBR:IC_ADS125H01IRHBT"
+		(property "Footprint" "audio-codec:IC_ADS125H01IRHBT"
 			(at 200.66 81.28 0)
 			(effects
@@
 			)
 		)
-		(property "Footprint" "MegaCastle:MegaCastle2x11-Module-I17.7x23.1-MBFFFFC-PANEL-NIBBLE"
+		(property "Footprint" "MegaCastle:MegaCastle2x11-Module-I22.0x23.1-MBFFFFC-SPAREPAD"
 			(at 100.33 146.05 0)
 			(effects
@@
 			)
 		)
-		(property "Footprint" "BGA9C50P3X3_187X165X66N"
+		(property "Footprint" "audio-codec:BGA9C50P3X3_187X165X66N"
 			(at 85.09 64.77 0)
 			(effects
@@
 		)
 	)
+	(embedded_fonts no)
 )
