File: modules/cellular-modem/cellular-modem.kicad_pcb (KiCad board)
At the start: 4 copper layers, 42.8 x 71.1 mm, 23 parts, among them J1 MM60-mini-PCIe, J2 MM60-EZH059-B5-R650, U1 TXV0108RGYR, U2 TXV0108RGYR, U3 TXV0108RGYR, U4 TPS631000DRLR, U5 TPS631000DRLR

Commit message: Updating cellular-modem
Routing:
- net /COEX_UART_TX_1V8_OUT: track 29.4 -> 28.5 mm
- net /UART_TX_1V8_OUT: track 24.5 -> 23.7 mm
- net GND: vias 113 -> 132
