File: modules/te0725-carrier/te0725-carrier.kicad_pcb (KiCad board)
At the start: 2 copper layers, 2 parts, among them J1 Conn_02x25_Odd_Even, J2 Conn_02x25_Odd_Even

Commit message: route etc on TE0725 carrier module
Parts:
- added M1: ~, MegaCastle:MegaCastle2x52-Module-I42.0x127.3-M1, F.Cu at (65.5, 109.5)
Connections:
- J1 pad 1: unconnected-(J1-Pin_1-Pad1) -> J1_1
- J1 pad 10: unconnected-(J1-Pin_10-Pad10) -> J1_10
- J1 pad 11: unconnected-(J1-Pin_11-Pad11) -> J1_11
- J1 pad 12: unconnected-(J1-Pin_12-Pad12) -> J1_12
- J1 pad 13: unconnected-(J1-Pin_13-Pad13) -> J1_13
- J1 pad 14: unconnected-(J1-Pin_14-Pad14) -> J1_14
- J1 pad 15: unconnected-(J1-Pin_15-Pad15) -> J1_15
- J1 pad 16: unconnected-(J1-Pin_16-Pad16) -> J1_16
- J1 pad 17: unconnected-(J1-Pin_17-Pad17) -> J1_17
- J1 pad 18: unconnected-(J1-Pin_18-Pad18) -> J1_18
- J1 pad 19: unconnected-(J1-Pin_19-Pad19) -> J1_19
- J1 pad 2: unconnected-(J1-Pin_2-Pad2) -> J1_1
- J1 pad 20: unconnected-(J1-Pin_20-Pad20) -> J1_20
- J1 pad 21: unconnected-(J1-Pin_21-Pad21) -> J1_21
- J1 pad 22: unconnected-(J1-Pin_22-Pad22) -> J1_22
- J1 pad 23: unconnected-(J1-Pin_23-Pad23) -> J1_23
- J1 pad 24: unconnected-(J1-Pin_24-Pad24) -> J1_24
- J1 pad 25: unconnected-(J1-Pin_25-Pad25) -> J1_25
- J1 pad 26: unconnected-(J1-Pin_26-Pad26) -> J1_26
- J1 pad 27: unconnected-(J1-Pin_27-Pad27) -> J1_27
- J1 pad 28: unconnected-(J1-Pin_28-Pad28) -> J1_28
- J1 pad 29: unconnected-(J1-Pin_29-Pad29) -> J1_29
- J1 pad 3: unconnected-(J1-Pin_3-Pad3) -> J1_3
- J1 pad 30: unconnected-(J1-Pin_30-Pad30) -> J1_30
- J1 pad 31: unconnected-(J1-Pin_31-Pad31) -> J1_31
- J1 pad 32: unconnected-(J1-Pin_32-Pad32) -> J1_32
- J1 pad 33: unconnected-(J1-Pin_33-Pad33) -> J1_33
- J1 pad 34: unconnected-(J1-Pin_34-Pad34) -> J1_34
- J1 pad 35: unconnected-(J1-Pin_35-Pad35) -> J1_35
- J1 pad 36: unconnected-(J1-Pin_36-Pad36) -> J1_36
- J1 pad 37: unconnected-(J1-Pin_37-Pad37) -> J1_37
- J1 pad 38: unconnected-(J1-Pin_38-Pad38) -> J1_38
- J1 pad 39: unconnected-(J1-Pin_39-Pad39) -> J1_39
- J1 pad 4: unconnected-(J1-Pin_4-Pad4) -> J1_4
- J1 pad 40: unconnected-(J1-Pin_40-Pad40) -> J1_40
- J1 pad 41: unconnected-(J1-Pin_41-Pad41) -> J1_41
- J1 pad 42: unconnected-(J1-Pin_42-Pad42) -> J1_42
- J1 pad 43: unconnected-(J1-Pin_43-Pad43) -> J1_43
- J1 pad 44: unconnected-(J1-Pin_44-Pad44) -> J1_44
- J1 pad 45: unconnected-(J1-Pin_45-Pad45) -> J1_45
- J1 pad 46: unconnected-(J1-Pin_46-Pad46) -> J1_46
- J1 pad 47: unconnected-(J1-Pin_47-Pad47) -> J1_47
- J1 pad 48: unconnected-(J1-Pin_48-Pad48) -> J1_48
- J1 pad 49: unconnected-(J1-Pin_49-Pad49) -> J1_1
- J1 pad 5: unconnected-(J1-Pin_5-Pad5) -> J1_46
- J1 pad 50: unconnected-(J1-Pin_50-Pad50) -> J1_1
- J1 pad 6: unconnected-(J1-Pin_6-Pad6) -> J1_45
- J1 pad 7: unconnected-(J1-Pin_7-Pad7) -> J1_7
- J1 pad 8: unconnected-(J1-Pin_8-Pad8) -> J1_8
- J1 pad 9: unconnected-(J1-Pin_9-Pad9) -> J1_9
- J2 pad 1: unconnected-(J2-Pin_1-Pad1) -> J1_1
- J2 pad 10: unconnected-(J2-Pin_10-Pad10) -> J2_10
- J2 pad 11: unconnected-(J2-Pin_11-Pad11) -> J2_11
- J2 pad 12: unconnected-(J2-Pin_12-Pad12) -> J2_12
- J2 pad 13: unconnected-(J2-Pin_13-Pad13) -> J2_13
- J2 pad 14: unconnected-(J2-Pin_14-Pad14) -> J2_14
- J2 pad 15: unconnected-(J2-Pin_15-Pad15) -> J2_15
- J2 pad 16: unconnected-(J2-Pin_16-Pad16) -> J2_16
- J2 pad 17: unconnected-(J2-Pin_17-Pad17) -> J2_17
- J2 pad 18: unconnected-(J2-Pin_18-Pad18) -> J2_18
- J2 pad 19: unconnected-(J2-Pin_19-Pad19) -> J2_19
- J2 pad 2: unconnected-(J2-Pin_2-Pad2) -> J1_1
- J2 pad 20: unconnected-(J2-Pin_20-Pad20) -> J2_20
- J2 pad 21: unconnected-(J2-Pin_21-Pad21) -> J2_21
- J2 pad 22: unconnected-(J2-Pin_22-Pad22) -> J2_22
- J2 pad 23: unconnected-(J2-Pin_23-Pad23) -> J2_23
- J2 pad 24: unconnected-(J2-Pin_24-Pad24) -> J2_24
- J2 pad 25: unconnected-(J2-Pin_25-Pad25) -> J2_25
- J2 pad 26: unconnected-(J2-Pin_26-Pad26) -> J2_26
- J2 pad 27: unconnected-(J2-Pin_27-Pad27) -> J2_27
- J2 pad 28: unconnected-(J2-Pin_28-Pad28) -> J2_28
- J2 pad 29: unconnected-(J2-Pin_29-Pad29) -> J2_29
- J2 pad 3: unconnected-(J2-Pin_3-Pad3) -> J2_3
- J2 pad 30: unconnected-(J2-Pin_30-Pad30) -> J2_30
- J2 pad 31: unconnected-(J2-Pin_31-Pad31) -> J2_31
- J2 pad 32: unconnected-(J2-Pin_32-Pad32) -> J2_32
- J2 pad 33: unconnected-(J2-Pin_33-Pad33) -> J2_33
- J2 pad 34: unconnected-(J2-Pin_34-Pad34) -> J2_34
- J2 pad 35: unconnected-(J2-Pin_35-Pad35) -> J2_35
- J2 pad 36: unconnected-(J2-Pin_36-Pad36) -> J2_36
- J2 pad 37: unconnected-(J2-Pin_37-Pad37) -> J2_37
- J2 pad 38: unconnected-(J2-Pin_38-Pad38) -> J2_38
- J2 pad 39: unconnected-(J2-Pin_39-Pad39) -> J2_39
- J2 pad 4: unconnected-(J2-Pin_4-Pad4) -> J2_4
- J2 pad 40: unconnected-(J2-Pin_40-Pad40) -> J2_40
- J2 pad 41: unconnected-(J2-Pin_41-Pad41) -> J2_41
- J2 pad 42: unconnected-(J2-Pin_42-Pad42) -> J2_42
- J2 pad 43: unconnected-(J2-Pin_43-Pad43) -> J2_43
- J2 pad 44: unconnected-(J2-Pin_44-Pad44) -> J2_44
- J2 pad 45: unconnected-(J2-Pin_45-Pad45) -> J1_45
- J2 pad 46: unconnected-(J2-Pin_46-Pad46) -> J1_46
- J2 pad 47: unconnected-(J2-Pin_47-Pad47) -> J2_47
- J2 pad 48: unconnected-(J2-Pin_48-Pad48) -> J2_48
- J2 pad 49: unconnected-(J2-Pin_49-Pad49) -> J1_1
- J2 pad 5: unconnected-(J2-Pin_5-Pad5) -> J1_46
- J2 pad 50: unconnected-(J2-Pin_50-Pad50) -> J1_1
- J2 pad 6: unconnected-(J2-Pin_6-Pad6) -> J1_45
- J2 pad 7: unconnected-(J2-Pin_7-Pad7) -> J2_7
- J2 pad 8: unconnected-(J2-Pin_8-Pad8) -> J2_8
- J2 pad 9: unconnected-(J2-Pin_9-Pad9) -> J2_9
Routing:
- net J1_1: track 0.00 -> 204.4 mm
- net J1_46: track 0.00 -> 183.4 mm, vias 0 -> 1
- net J1_45: track 0.00 -> 166.1 mm
- net J1_4: track 0.00 -> 134.1 mm
- net J1_8: track 0.00 -> 123.0 mm
- net J1_10: track 0.00 -> 117.3 mm
- net J2_8: track 0.00 -> 116.4 mm
- net J1_12: track 0.00 -> 111.3 mm
- net J2_10: track 0.00 -> 110.3 mm
- net J2_12: track 0.00 -> 104.9 mm
- net J1_14: track 0.00 -> 104.6 mm
- net J1_16: track 0.00 -> 100.0 mm
- net J2_14: track 0.00 -> 98.8 mm
- net J2_16: track 0.00 -> 93.8 mm
- net J1_18: track 0.00 -> 93.7 mm
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Other:
- board outline added: 42 x 132.1 mm
